File: hardware/eagle/DWM1000_Feather.sch (EAGLE design)
At the start: 41 parts, among them J1 DX07B024JJ3R1600, J4 20021221-00010C4LF, SW1 SPST_TACT-KMR2, U1 ATSAMD21G-M, U2 MCP73831, U3 DWM1000, U4 AP2112K-3.3TRG1, Y1 FC-135_32.7680KA-A0

Commit message: Version 1.1 update. BRD is INCOMPLETE
Parts:
- removed D5: BLUE, SparkFun-LED:LED0603
- removed J1: DX07B024JJ3R1600, DX07B024JJ3R1600:DX07B024JJ3R1600
- removed R10: 10K, SparkFun-Resistors:RESISTOR0603
- removed TP6: TEST-POINT2, SparkFun-Connectors:TEST-POINT2
- added R7: 100K, SparkFun-Resistors:RESISTOR0603
- added R8: YC124-JR-07330RL, YC124-JR-07330RL:YC124-JR-07330RL
- added TP2: TEST-POINT3, SparkFun-Connectors:TEST-POINT3
- D1: value ORANGE -> (none); device SparkFun-LED:LED0603 -> adafruit:DIODE_SOD-123FL
- D2: value (none) -> ASMT-YTD7-0AA02; device adafruit:DIODE_SOD-123FL -> ASMT-YTD7-0AA02:ASMT-YTD7-0AA02
- J4: value 20021221-00010C4LF -> USB4110-GF-A; device 20021221-00010C4LF:20021221-00010C4LF -> USB4110-GF-A:USB4110-GF-A
- JP1: value BATT_DETECT -> DWM_3V3
- JP2: value DWM_3V3 -> 20021221-00010C4LF; device SparkFun-Jumpers:JUMPER-SMT_2_NC_TRACE_SILK -> 20021221-00010C4LF:20021221-00010C4LF
- R4: value 1K -> 5K1
- R9: value 330 -> 10K
- TP1, TP3, TP4, TP5: value TEST-POINT2 -> TEST-POINT3; device SparkFun-Connectors:TEST-POINT2 -> SparkFun-Connectors:TEST-POINT3
- U2: value MCP73831 -> MCP73832
Connections:
- removed net CC1: J1.CC1, R1.2, TP3.1
- removed net CC2: J1.CC2, R2.2, TP4.1
- removed net DWM_WU: U3.WAKEUP
- removed net N$9: D5.A, R9.1
- removed net RX_LED: U3.GPIO2
- removed net TX_LED: U3.GPIO3
- new net BATT_S: R4.2, U1.PA28, U2.STAT
- new net BATT_V: R3.2, R5.1, U1.PB03(AIN11/SER5:1)
- new net N$1: D2.B_A, R8.5
- new net N$10: J4.CC2, R2.2
- new net N$8: J4.CC1, R1.2
- new net RGB_B: R8.4, U1.PB22(SER5:2+)
- new net RGB_G: R8.3, U1.PB23(SER5:3+)
- new net RGB_R: R8.2, U1.PA27
- net 3.3V: now also JP1.2, JP2.1, R4.1; no longer J4.1, JP2.2
- net D+: now also J4.DP1, J4.DP2, TP1.1; no longer J1.DA+, J1.DB+
- net D-: now also J4.DN1, J4.DN2, TP2.1; no longer J1.DA-, J1.DB-
- net D13: no longer R9.2
- net D2: no longer TP5.1
- net D3: now also R7.2; no longer TP6.1
- net D9: no longer JP1.2
- net DWM_3V3: now also JP1.1, TP5.1; no longer JP2.1, TP1.1
- net EN: now also R9.2; no longer R10.2
- net GND: now also D2.B_C, D2.G_C, D2.R_C, J4.GND, JP2.3, JP2.5, JP2.9, R5.2, R7.1; no longer D5.C, J1.GNDA, J1.GNDB, J1.SHIELD, J4.3, J4.5, J4.9, R3.1
- net N$3: now also D2.G_A, R8.6; no longer D1.C, R4.1
- net N$4: now also R8.7, R8.8; no longer R4.2, U2.STAT
- net N$5: now also D2.R_A, R8.1; no longer JP1.1, R3.2, R5.1
- net SWCLK: now also JP2.4, TP4.1; no longer J4.4
- net SWDIO: now also JP2.2, TP3.1; no longer J4.2
- net V_BATT: now also D1.A, R3.1; no longer D2.A, R5.2
- net V_USB: now also D1.C, J4.VBUS, R9.1; no longer D1.A, D2.C, J1.A_VBUS, J1.B_VBUS, R10.1
Other:
- note added: "NOTE: MCP73832 is open-drain. STAT pin is pulled-up to 3V3 for reading by micro"
- note added: "Prototyping Corner"
- moved on the sheet: C5, CN1, JP1, R1, R2, R3, R4, R5, R6, R9, TP1, TP3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

Commit message: Updated for version 1.1
Parts:
- removed JP2: 20021221-00010C4LF, 20021221-00010C4LF:20021221-00010C4LF
- added J1: USB4110-GF-A, USB4110-GF-A:USB4110-GF-A
- C1, C4, C5, C6, C7, C8, C9: device SparkFun-Capacitors:10UF-0603-6.3V-20% -> SparkFun-Capacitors-edit:10UF-POLAR-0603-6.3V-20%(TANT)
- J4: value USB4110-GF-A -> 20021221-00010C4LF; device USB4110-GF-A:USB4110-GF-A -> 20021221-00010C4LF:20021221-00010C4LF
- LOGO1: value OSHW-LOGOL -> OSHW-LOGOS; device SparkFun-Aesthetics:OSHW-LOGOL -> SparkFun-Aesthetics:OSHW-LOGOS
- R9: value 10K -> 100K
Connections:
- net 3.3V: now also J4.1; no longer JP2.1
- net D+: now also J1.DP1, J1.DP2; no longer J4.DP1, J4.DP2
- net D-: now also J1.DN1, J1.DN2; no longer J4.DN1, J4.DN2
- net GND: now also J1.GND, J4.3, J4.5, J4.9; no longer J4.GND, JP2.3, JP2.5, JP2.9
- net N$10: now also J1.CC2; no longer J4.CC2
- net N$8: now also J1.CC1; no longer J4.CC1
- net SWCLK: now also J4.4; no longer JP2.4
- net SWDIO: now also J4.2; no longer JP2.2
- net V_USB: now also J1.VBUS; no longer J4.VBUS
Other:
- note added: "Licensed under CERN OHL v1.2"
- note removed: "SPFDB"
